File: Watchy.sch (KiCad schematic (older format))
At the start: 55 parts, among them J1 FPC24(0.5MM), J2 Micro USB, J3 Battery, M1 Vibration_Motor, Q1 AO3400A, Q2 UMH3N, Q4 CJ2301, Q5 S8050, SW1 BTN, SW2 BTN, SW3 BTN, SW4 BTN, U1 ESP32-PICO-D4, U2 ME6211C33M5G-N, U3 CP2104, U4 BMA423, U5 TP4054, U6 DS3231MZ

Commit message: added or replaced parts and altered borad outline
Parts:
- removed C10, C2, C5, C6, C7, C8, C9: 1uF/50V, Capacitor_SMD:C_0603_1608Metric, symbol Device:C
- removed C3, C4: 4.7uF/50V, Capacitors_SMD:C_0805, symbol Device:C
- removed D1, D2, D3: MBR0530, Diodes_SMD:D_SOD-123, symbol Device:D
- removed J1: FPC24(0.5MM), Watchy:24_Pins_0.5mm_Pitch_ZIF_Connector_UP, symbol Connector_Generic:Conn_01x24
- removed L1: 10uH 1A, Inductors:Inductor_Taiyo-Yuden_NR-40xx, symbol Device:L
- removed Q1: AO3400A, TO_SOT_Packages_SMD:SOT-23, symbol Transistor_FET:DMN3042L
- removed R8: 10K, Resistors_SMD:R_0402, symbol Device:R
- removed R9: 3, Resistors_SMD:R_0402, symbol Device:R
- removed U6: DS3231MZ, Housings_SOIC:SOIC-8_3.9x4.9mm_Pitch1.27mm, symbol Timer_RTC:DS3231MZ
- added J1: 503480-0400, Watchy:MOLEX_503480-0400, symbol Watchy:503480-0400
- added J4: FH33-10S-0.5SH_10_, Watchy:FH3310S05SH10, symbol Watchy:FH33-10S-0.5SH_10_
- added U10: BME280, Package_LGA:Bosch_LGA-8_2.5x2.5mm_P0.65mm_ClockwisePinNumbering, symbol Sensor:BME280
- added U7: MX25R3235FZNxx1, Package_SON:WSON-8-1EP_6x5mm_P1.27mm_EP3.4x4mm, symbol Memory_Flash:MX25R3235FZNxx1
- added U8: L76-L, Watchy:XCVR_L76-L, symbol Watchy:L76-L
- added U9: IIS2MDCTR, Watchy:IIS2MDCTR, symbol Watchy:IIS2MDCTR
- added Y1: RV-8523-C3-TA-QC-020, Watchy:RV8523C3TAQC020, symbol Watchy:RV-8523-C3-TA-QC-020
Connections:
- net labels removed: +3.3V, GDR, PREVGH, PREVGL, RESE
- wire segments 39 -> 35
- no-connect marks 40 -> 35
Other:
- moved on the sheet: U4
