File: Watchy.sch (KiCad schematic (older format))
At the start: 44 parts, among them J1 503480-0400, J2 Micro USB, J3 Battery, J4 FH33-10S-0.5SH_10_, M1 Vibration_Motor, Q2 UMH3N, Q4 CJ2301, Q5 S8050, SW1 BTN, SW2 BTN, SW3 BTN, SW4 BTN, U1 ESP32-PICO-D4, U10 BME280, U2 ME6211C33M5G-N, U3 CP2104, U4 BMA423, U5 TP4054, U7 MX25R3235FZNxx1, U8 L76-L, U9 IIS2MDCTR, Y1 RV-8523-C3-TA-QC-020

Commit message: version 0 production
Parts:
- removed U8: L76-L, Watchy:XCVR_L76-L, symbol Watchy:L76-L
- added C10, C13, C2, C4, C5, C8: 100nF, Capacitor_SMD:C_0603_1608Metric, symbol Device:C
- added C3: 1uF, Capacitor_SMD:C_0603_1608Metric, symbol Device:C
- added C6, C7: 220nF, Capacitor_SMD:C_0603_1608Metric, symbol Device:C
- added C9: 10uF/50V, Capacitor_SMD:C_0805_2012Metric, symbol Device:C
- added IC1: L76L-M33, Watchy:L76, symbol Watchy:L76-M33
- added J5: U.FL-R-SMT(01), Watchy:HRS_U.FL-R-SMT(01), symbol Watchy:U.FL-R-SMT(01)
- added J6: Conn_01x04_Female, Connector_PinSocket_1.00mm:PinSocket_1x04_P1.00mm_Vertical, symbol Connector:Conn_01x04_Female
- added JP1: SolderJumper_3_Open, Jumper:SolderJumper-3_P1.3mm_Open_Pad1.0x1.5mm, symbol Jumper:SolderJumper_3_Open
- added R8: 3.5K, Resistor_SMD:R_0402_1005Metric, symbol Device:R
- added R9: 10K, Resistor_SMD:R_0402_1005Metric, symbol Device:R
- added U6: CAT4004AHU2-GT3, Watchy:CAT4004AHU2-GT3, symbol Watchy:CAT4004AHU2-GT3
- added U8: LTR-303ALS-01, OptoDevice:Lite-On_LTR-303ALS-01, symbol Sensor_Optical:LTR-303ALS-01
- D4: LCSC (none) -> C77336; MPN (none) -> MBR0530
- D5: LCSC (none) -> C2286; MPN (none) -> LTST-C190KRKT
- D6: LCSC (none) -> C433392; MPN (none) -> 1N4001
- J1: LCSC (none) -> C563965; MPN (none) -> 503480-0400
- J2: LCSC (none) -> C91146; LCSC Alt (none) -> C145792; MPN (none) -> U-F-M5DD-Y-L
- J3: LCSC (none) -> C189700; MPN (none) -> 532610271
- J4: value FH33-10S-0.5SH_10_ -> FH33-10S-0.5SH(10); MPN (none) -> FH33-10S-0.5SH(10); Manufacturer_Part_Number FH33-10S-0.5SH(10) -> (none)
- Q2: LCSC (none) -> C62892; MPN (none) -> UMH3N
- Q4: LCSC (none) -> C8547; MPN (none) -> CJ2301
- Q5: LCSC (none) -> C2146; MPN (none) -> S8050
- R1, R10, R12, R13, R14, R15, R16, R17, R2, R3, R4, R5, R6, R7: footprint Resistors_SMD:R_0402 -> Resistor_SMD:R_0402_1005Metric
- SW1, SW2, SW3, SW4: LCSC (none) -> C136662; MPN (none) -> K2-1114SA-A4SW-06
- U1: LCSC (none) -> C193707; MPN (none) -> ESP32-PICO-D4
- U10: LCSC (none) -> C92489; MPN (none) -> BME280
- U2: LCSC (none) -> C82942; MPN (none) -> ME6211C33M5G-N
- U3: LCSC (none) -> C430013; MPN (none) -> CP2104-F03-GM
- U4: Field4 Bosch Sensortec -> (none); LCSC (none) -> C189517; MF (none) -> Bosch Sensortec; MPN (none) -> BMA423
- U5: LCSC (none) -> C32574; MPN (none) -> TP4054
- U7: value MX25R3235FZNxx1 -> MX25L25645GZN-10G; LCSC (none) -> C2802981; MPN (none) -> MX25L25645GZN-10G
- U9: LCSC (none) -> C2655002; MPN (none) -> IIS2MDCTR
- Y1: MPN (none) -> RV-8523-C3-TA-QC-020; Manufacturer_Part_Number RV-8523-C3-TA-QC-020 -> (none)
Connections:
- net labels added: ATGM, BL_PWM, EXTCOM, FLASH_CLK, FLASH_CS, FLASH_MISO, FLASH_MOSI, GPS_FORCE_ON, GPS_RX, GPS_TX, INT_ACC1, INT_ACC2, INT_ALS, INT_RTC, LCD_CLK, LCD_CS, LCD_EN, LCD_MOSI, QUECTEL, RF
- net labels removed: ACC_INT_1, ACC_INT_2, BUSY, DC, MOSI, RES, RTC_INT, SCK, SS
- wire segments 35 -> 77
- no-connect marks 35 -> 45
Other:
- note added: "FLASH"
- note added: "GPS"
- note added: "MLCD Driver"
- note added: "Sensors"
- note removed: "Accelerometer"
- note removed: "E-Paper Driver"
- moved on the sheet: J1, J4, U10, U7, U9, Y1

Commit message: v0 PCBWay final version
Changed lines of the file:
@@
 Vibration Motor
 Wire Notes Line
-	3270 6645 3270 7795
+	3120 6650 3120 7800
 $Comp
 L Device:LED D5
@@
 Text GLabel 6265 2165 0    50   Input ~ 0
 ATGM
+Wire Notes Line
+	4590 6640 4590 7790
+Wire Notes Line
+	4590 7790 4600 7790
 $EndSCHEMATC
